File: panels/mod1-tap-tempo/mod1-tap-tempo.kicad_pcb (KiCad board)
At the start: 2 copper layers, 19.8 x 128.5 mm, 0 parts

Commit message: move vcvrack, update faceplates
Other:
- board text added: "1x output"
- board text added: "Div 1"
- board text added: "Div 2"
- board text added: "Mult 1"
- board text added: "tap tempo (4x)"
- board text added: "| TAP TEMPO |"
- board text removed: "1x"
- board text removed: "Div"
- board text removed: "Mult"
- board text removed: "TAP TEMPO"
- board text removed: "Var"
- board text removed: "tap"
