File: panels/mod2-breakbeats/mod2-breakbeats.kicad_pcb (KiCad board)
At the start: 2 copper layers, 19.8 x 128.5 mm, 0 parts

Commit message: move vcvrack, update faceplates
Other:
- board text added: "BREAKBEATS"
- board text removed: "BREAKBEAT"
- board text removed: "CV"
