File: panels/mod2-flux/mod2-flux.kicad_pcb (KiCad board)
At the start: 2 copper layers, 19.8 x 128.5 mm, 0 parts

Commit message: move vcvrack, update faceplates
Other:
- board text added: "- modal - karplus - white - pink - s&h - lorenz - drone"
- board text added: "Character"
- board text added: "Freq / Pitch"
- board text added: "mode select"
- board text added: "trigger"
- board text added: "| FLUX |"
- board text removed: "CV"
- board text removed: "FLUX"
- board text removed: "Freq"
- board text removed: "mode"
