File: panels/mod2-fm_drum/mod2-fm_drum.kicad_pcb (KiCad board)
At the start: 2 copper layers, 19.8 x 128.5 mm, 0 parts

Commit message: move vcvrack, update faceplates
Other:
- board text added: "1 | 2"
- board text added: "Pitch | Decay"
- board text added: "on = 2"
- board text added: "| FM DRUM |"
- board text removed: "CV"
- board text removed: "FM DRUM"
- board text removed: "Pitch"
- board text removed: "mode"
