File: panels/mod2-hihat/mod2-hihat.kicad_pcb (KiCad board)
At the start: 2 copper layers, 19.8 x 128.5 mm, 0 parts

Commit message: move vcvrack, update faceplates
Other:
- board text added: "Frequency"
- board text added: "env out"
- board text added: "tap = trig long = type"
- board text added: "| HIHAT |"
- board text removed: "CV"
- board text removed: "HIHAT"
- board text removed: "env"
- board text removed: "type"
