File: panels/mod2-kick/mod2-kick.kicad_pcb (KiCad board)
At the start: 2 copper layers, 19.8 x 128.5 mm, 0 parts

Commit message: move vcvrack, update faceplates
Other:
- board text added: "1 | 2 save"
- board text added: "Clip | End"
- board text added: "Envelope"
- board text added: "Pitch | Start"
- board text added: "on = 2"
- board text removed: "CV"
- board text removed: "Clip"
- board text removed: "Pitch"
- board text removed: "env"
- board text removed: "param"
