File: panels/mod2-radio/mod2-radio.kicad_pcb (KiCad board)
At the start: 2 copper layers, 19.8 x 128.5 mm, 0 parts

Commit message: move vcvrack, update faceplates
Other:
- board text added: "Direction"
- board text added: "output"
- board text added: "trigger"
- board text added: "| RADIO |"
- board text removed: "CV"
- board text removed: "Dir"
- board text removed: "RADIO"
- board text removed: "trig"
