File: panels/mod2-sample/mod2-sample.kicad_pcb (KiCad board)
At the start: 2 copper layers, 19.8 x 128.5 mm, 0 parts

Commit message: move vcvrack, update faceplates
Other:
- board text added: "output"
- board text added: "trigger"
- board text added: "| SAMPLE |"
- board text removed: "CV"
- board text removed: "SAMPLE"
- board text removed: "trig"
