File: panels/mod2-spiral/mod2-spiral.kicad_pcb (KiCad board)
At the start: 2 copper layers, 19.8 x 128.5 mm, 0 parts

Commit message: move vcvrack, update faceplates
Other:
- board text added: "Frequency"
- board text added: "V/Oct"
- board text added: "mode select"
- board text added: "on = dir"
- board text added: "short = cycle long = dir"
- board text added: "| SPIRALS |"
- board text removed: "CV"
- board text removed: "Freq"
- board text removed: "SPIRAL"
- board text removed: "dir"
- board text removed: "mode"
