File: panels/mod2-square_vco/mod2-square_vco.kicad_pcb (KiCad board)
At the start: 2 copper layers, 19.8 x 128.5 mm, 0 parts

Commit message: move vcvrack, update faceplates
Other:
- board text added: "SQUARE VCO"
- board text added: "chiptune on/off"
- board text added: "on = chip"
- board text removed: "SQ VCO"
- board text removed: "chip"
- board text removed: "mode"
