File: panels/fm-output/fm-output.kicad_pcb (KiCad board)
At the start: 2 copper layers, 40.3 x 128.5 mm, 0 parts

Commit message: fixing licensing, updating fm-out
Other:
- board text added: "In Left"
- board text added: "In Right"
- board text added: "Line Left"
- board text added: "Line Right"
- board text removed: "In L"
- board text removed: "In R"
- board text removed: "L"
- board text removed: "R"
